Commit message: [Jl+bar version] first commit

File: chr_description/urdf/chr.urdf (robot description, URDF)
Before this commit: robot cone_harvest_robot, 11 links, 10 joints
Links:
- removed link arm_link2
- removed link arm_link3
- removed link arm_link4
- removed link tcp
- link arm_link1: geometry visual cylinder length=0.333 radius=0.01
Joints:
- removed joint J2
- removed joint J3
- removed joint arm_link3_to_link4
- removed joint tcp_fixed
- joint J1: axis 0 0 1 -> 0 1 0; limit lower=-1.5708 upper=1.5708 effort=10 velocity=1 -> lower=0 upper=1.5708 effort=10 velocity=1; origin xyz=0 0 0.04475 rpy=-1.5708 -1.5708 0 -> xyz=0 0 0.04475 rpy=0 0 0
